File: PCB/Sportify Playdeck.kicad_sch (KiCad schematic)
At the start: 6 parts, among them J1 Conn_01x04_Pin, SW1 SW_Push, SW2 SW_Push, SW3 SW_Push, SW4 SW_Push, U1 MOUDLE-SEEEDUINO-XIAO

Commit message: updated the schematics, assembly file and firmware
Connections:
- net at SW1.2, SW2.2, SW3.2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: now also J1.1 (Pin_1); no longer J1.2 (Pin_2)
- net at U1.12 (3V3): now also J1.2 (Pin_2); no longer J1.1 (Pin_1)
Changed lines of the file:
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@@
 		(color 0 0 0 0)
 	)
-	(bus_entry
-		(at 176.53 77.47)
-		(size 2.54 2.54)
+	(wire
+		(pts
+			(xy 186.69 60.96) (xy 177.8 60.96)
+		)
 		(stroke
 			(width 0)
@@
 	(wire
 		(pts
-			(xy 181.61 53.34) (xy 166.37 53.34)
+			(xy 166.37 53.34) (xy 186.69 53.34)
 		)
 		(stroke
@@
 	(wire
 		(pts
+			(xy 184.15 58.42) (xy 177.8 58.42)
+		)
+		(stroke
+			(width 0)
+			(type default)
+		)
+	)
+	(wire
+		(pts
 			(xy 109.22 96.52) (xy 109.22 101.6)
 		)
@@
 	(wire
 		(pts
+			(xy 186.69 53.34) (xy 186.69 60.96)
+		)
+		(stroke
+			(width 0)
+			(type default)
+		)
+	)
+	(wire
+		(pts
 			(xy 102.87 68.58) (xy 92.71 68.58)
 		)
@@
 	(wire
 		(pts
+			(xy 184.15 82.55) (xy 184.15 58.42)
+		)
+		(stroke
+			(width 0)
+			(type default)
+		)
+	)
+	(wire
+		(pts
 			(xy 120.65 76.2) (xy 97.79 76.2)
 		)
@@
 	(wire
 		(pts
-			(xy 184.15 82.55) (xy 184.15 60.96)
-		)
-		(stroke
-			(width 0)
-			(type default)
-		)
-	)
-	(wire
-		(pts
 			(xy 130.81 85.09) (xy 130.81 95.25)
 		)
@@
 	(wire
 		(pts
-			(xy 181.61 58.42) (xy 181.61 53.34)
-		)
-		(stroke
-			(width 0)
-			(type default)
-		)
-	)
-	(wire
-		(pts
 			(xy 116.84 77.47) (xy 95.25 77.47)
 		)
@@
 	(wire
 		(pts
-			(xy 177.8 58.42) (xy 181.61 58.42)
-		)
-		(stroke
-			(width 0)
-			(type default)
-		)
-	)
-	(wire
-		(pts
 			(xy 97.79 76.2) (xy 97.79 60.96)
 		)
@@
 		(pts
 			(xy 120.65 85.09) (xy 120.65 76.2)
-		)
-		(stroke
-			(width 0)
-			(type default)
-		)
-	)
-	(wire
-		(pts
-			(xy 177.8 60.96) (xy 184.15 60.96)
 		)
 		(stroke
@@
 		(property "Value" "Conn_01x04_Pin"
 			(at 173.355 55.88 0)
-			(show_name no)
-			(do_not_autoplace no)
+			(hide yes)
+			(show_name no)
+			(do_not_autoplace no)
